File: board/LX-15D-upgrade.kicad_pcb (KiCad board)
At the start: 2 copper layers, 19 x 29 mm, 36 parts, among them J1 M+, J2 M-, J3 IN-1, J4 IN-2, J5 SWD, U1 DRV8801A-Q1, U2 AS5600, U3 MPU-6050, U4 STM32L011F4Px, U5 AP7383-W5-3V3

Commit message: Add power decoupling capacitor
Parts:
- added C5: 47U, Capacitor_Tantalum_SMD:CP_EIA-6032-28_Kemet-C, F.Cu at (148.2, 106.8)
- C6: moved to B.Cu
- moved C6 1.79 mm to (146.9, 107.0)
- moved C13 0.15 mm to (142.4, 94.6)
- moved C14 0.15 mm to (145.8, 94.6)
- moved R1 0.11 mm to (151.7, 103.9)
- moved C2 0.05 mm to (151.7, 108.8)
- moved C3 0.05 mm to (151.7, 107.2)
Routing:
- net GND: track 62.9 -> 51.0 mm
- net PWR: track 27.5 -> 25.0 mm, vias 1 -> 2
- net VCC: track 28.5 -> 30.1 mm
- net Net-(D4-Pad1): vias 0 -> 1
- net Net-(D3-Pad1): vias 0 -> 1
- net Net-(D2-Pad1): vias 0 -> 1

Commit message: Final tweak
Parts:
- moved C6 0.38 mm to (147.2, 107.0)
Changed lines of the file:
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@@
   )
   (module Capacitor_SMD:C_0603_1608Metric_Pad1.05x0.95mm_HandSolder (layer B.Cu)
-    (at 146.875 107 180)
+    (at 147.25 107 180)
     (descr "Capacitor SMD 0603 (1608 Metric), square (rectangular) end terminal, IPC_7351 nominal with elongated pad for handsoldering. (Body size source: http://www.tortai-tech.com/upload/download/2011102023233369053.pdf), generated with kicad-footprint-generator")
     (tags "capacitor handsolder")
